File: forte-encoder-pcb.kicad_pcb (KiCad board)
At the start: 6 copper layers, 36.5 x 45 mm, 54 parts, among them J0 BM07B-SRSS-TB(LF)(SN), J1 Conn_01x01_Pin, J4 Conn_01x01_Pin, U2 STM32F103C8Tx, U3 MCP2542FD-E/MF, U4 MA732GQ-Z, U5 TPS629203DRLR, U6 TPS629203DRLR, Y1 CSTNE8M00G550000R0

Commit message: change port and rearange
Parts:
- removed J0: BM07B-SRSS-TB(LF)(SN), dash:BM07B-SRSS-TB
- added J2: BM07B-GHS-TBT, dash:JST_BM07B-GHS-TBT, F.Cu at (88.8, 113.5)
- TP_GND: renamed from TP GND
- moved SCK 19.0 mm to (116.2, 105.5)
- moved J8 15.7 mm to (98.7, 120.8)
- moved MISO 15.6 mm to (115.4, 107.9)
- moved J9 15.5 mm to (101.2, 120.4)
- moved J10 15.4 mm to (103.6, 119.6)
- moved J7 15.2 mm to (105.9, 118.4)
- moved CS 14.7 mm to (112.5, 105.9)
- moved MOSI 12.3 mm to (109.1, 101.7)
- moved C36 5.92 mm to (96.8, 110.0)
- moved C35 3.47 mm to (98.8, 110.0)
- moved U3 3.09 mm to (98.8, 115.1)
- moved D2 2.77 mm to (108.2, 116.0), turned to 180 degrees
- moved C29 1.10 mm to (104.3, 116.0), turned to 180 degrees
- renumbered CAN+ to J10, CAN+ to J7, - to J8, CAN- to J9
Routing:
- net /SCK: track 51.7 -> 28.3 mm, vias 2 -> 1
- net /CS: track 35.0 -> 11.9 mm, vias 2 -> 0
- net /MISO: track 34.3 -> 17.2 mm, vias 2 -> 1
- net /CAN-: track 66.2 -> 49.4 mm, vias 2 -> 0
- net /CAN+: track 61.7 -> 49.8 mm, vias 2 -> 0
- net /MOSI: track 33.2 -> 24.3 mm, vias 2 -> 1
- net +3.3V: track 88.9 -> 96.9 mm
- net +5V: track 31.3 -> 26.5 mm
- net /CAN_RX: track 16.2 -> 19.6 mm
- net /CAN_TX: track 10.00 -> 12.5 mm, vias 1 -> 2
- net GND: track 64.0 -> 62.7 mm
- net /TMS: track 14.0 -> 15.1 mm
- net /TCK: track 16.1 -> 16.9 mm
- net /USART_RX: track 30.0 -> 30.6 mm
Other:
- board text added: "CAN+"
- board text added: "CAN-"
- board text removed: "+"
- board text removed: "-"

Commit message: tiiny fix
Routing:
- net /MOSI: track 24.3 -> 16.1 mm
Changed lines of the file:
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@@
 	(segment
 		(start 107.4478 100.750001)
-		(end 108.497799 101.8)
+		(end 108.397799 101.7)
+		(width 0.2)
+		(layer "B.Cu")
+		(net "/MOSI")
+	)
+	(segment
+		(start 108.397799 101.7)
+		(end 109.1 101.7)
 		(width 0.2)
 		(layer "B.Cu")
@@
 	)
 	(segment
-		(start 108.497799 101.8)
-		(end 113.5 101.8)
-		(width 0.2)
-		(layer "B.Cu")
-		(net "/MOSI")
-	)
-	(segment
 		(start 115.1 109.2)
 		(end 115.05 109.25)
 		(width 0.2)
 		(layer "B.Cu")
-		(net "/MOSI")
-	)
-	(segment
-		(start 113.5 101.8)
-		(end 116.1 104.4)
-		(width 0.2)
-		(layer "B.Cu")
