File: forte-encoder-pcb.kicad_sch (KiCad schematic)
At the start: 54 parts, among them CN3(OUT)1 XT30(2+2)PB-M.G.B, J1 Conn_01x01_Pin, J10 Conn_01x01_Pin, J2 BM07B-GHS-TBT, J4 Conn_01x01_Pin, J7 Conn_01x01_Pin, J8 Conn_01x01_Pin, J9 Conn_01x01_Pin, U2 STM32F103C8Tx, U3 MCP2542FD-E/MF, U4 MA732GQ-Z, U5 TPS629203DRLR, U6 TPS629203DRLR, Y1 CSTNE8M00G550000R0

Commit message: fix TMS PA15->PA13
Connections:
- net TMS: now also U2.34 (PA13); no longer U2.38 (PA15)
Changed lines of the file:
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@@
-	)
-	(no_connect
-		(at 80.01 72.39)
 	)
 	(no_connect
@@
 	)
 	(no_connect
+		(at 74.93 72.39)
+	)
+	(no_connect
 		(at 95.25 36.83)
 	)
@@
 	(wire
 		(pts
-			(xy 74.93 72.39) (xy 74.93 82.55)
-		)
-		(stroke
-			(width 0)
-			(type default)
-		)
-	)
-	(wire
-		(pts
 			(xy 402.59 158.75) (xy 412.75 158.75)
 		)
@@
 		(pts
 			(xy 518.16 50.8) (xy 518.16 53.34)
+		)
+		(stroke
+			(width 0)
+			(type default)
+		)
+	)
+	(wire
+		(pts
+			(xy 80.01 72.39) (xy 80.01 82.55)
 		)
 		(stroke
@@
 		)
 	)
-	(label "TMS"
-		(at 74.93 82.55 90)
-		(effects
-			(font
-				(size 1.27 1.27)
-				(thickness 0.1588)
-			)
-			(justify left bottom)
-		)
-	)
 	(label "CS"
 		(at 57.15 177.8 0)
@@
 			)
 			(justify left bottom)
+		)
+	)
+	(label "TMS"
+		(at 80.01 82.55 90)
+		(effects
+			(font
+				(size 1.27 1.27)
+				(thickness 0.1588)
+			)
+			(justify left bottom)

Commit message: swap can
Connections:
- net CAN+: now also CN3(OUT)1.2; no longer CN3(OUT)1.1
- net CAN-: now also CN3(OUT)1.1; no longer CN3(OUT)1.2
Changed lines of the file:
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@@
-		)
-	)
-	(label "CAN+"
-		(at 402.59 156.21 0)
-		(effects
-			(font
-				(size 1.27 1.27)
-			)
-			(justify left bottom)
 		)
 	)
@@
 	)
 	(label "CAN-"
-		(at 402.59 158.75 0)
+		(at 402.59 156.21 0)
 		(effects
 			(font
@@
 		(effects
 			(font
+				(size 1.27 1.27)
+			)
+			(justify left bottom)
+		)
+	)
+	(label "CAN+"
+		(at 402.59 158.75 0)
+		(effects
+			(font

Commit message: more fix
Parts:
- removed TP_GND1: GND TestPoint, TestPoint:TestPoint_THTPad_D1.5mm_Drill0.7mm, symbol Connector:TestPoint
Changed lines of the file:
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@@
 	)
 	(junction
-		(at 416.56 82.55)
-		(diameter 0)
-		(color 0 0 0 0)
-	)
-	(junction
 		(at 320.04 39.37)
 		(diameter 0)
@@
 	(wire
 		(pts
-			(xy 416.56 78.74) (xy 416.56 82.55)
+			(xy 416.56 78.74) (xy 416.56 85.09)
 		)
 		(stroke
@@
 	(wire
 		(pts
-			(xy 416.56 82.55) (xy 416.56 85.09)
-		)
-		(stroke
-			(width 0)
-			(type default)
-		)
-	)
-	(wire
-		(pts
 			(xy 45.72 153.67) (xy 45.72 165.1)
 		)
@@
 					(unit 1)
 				)
-			)
-		)
-	)
-	(symbol
-		(lib_id "Connector:TestPoint")
-		(at 416.56 82.55 270)
-		(unit 1)
-		(body_style 1)
-		(exclude_from_sim no)
-		(in_bom yes)
-		(on_board yes)
-		(in_pos_files yes)
-		(dnp no)
-		(fields_autoplaced yes)
-		(property "Reference" "TP_GND1"
-			(at 421.64 81.2799 90)
-			(show_name no)
-			(do_not_autoplace no)
-			(effects
-				(font
-					(size 1.27 1.27)
-				)
-				(justify left)
-			)
-		)
-		(property "Value" "GND TestPoint"
-			(at 421.64 83.8199 90)
-			(show_name no)
-			(do_not_autoplace no)
-			(effects
-				(font
-					(size 1.27 1.27)
-				)
-				(justify left)
-			)
-		)
-		(property "Footprint" "TestPoint:TestPoint_THTPad_D1.5mm_Drill0.7mm"
-			(at 416.56 87.63 0)
-			(hide yes)
-			(show_name no)
-			(do_not_autoplace no)
-			(effects
-				(font
-					(size 1.27 1.27)
-				)
-			)
-		)
-		(property "Datasheet" ""
-			(at 416.56 87.63 0)
-			(hide yes)
-			(show_name no)
-			(do_not_autoplace no)
-			(effects
-				(font
-					(size 1.27 1.27)
-				)
-			)
-		)
-		(property "Description" "test point"
-			(at 416.56 82.55 0)
-			(hide yes)
-			(show_name no)
-			(do_not_autoplace no)
-			(effects
-				(font
-					(size 1.27 1.27)
-				)
-			)
-		)
-		(pin "1"
-		)
-		(instances
-			(project "forte-encoder-pcb"
-				(path "/4fd4f7f7-4e27-480c-b1ee-dc0730be04ca"
-					(reference "TP_GND1")
-					(unit 1)
-				)
